Commit message: Added transmission elements, still no wrist/gripper

File: urdf/roboarm.urdf.xacro (robot description, xacro)
@@ -136,4 +136,34 @@
 		<limit lower="${-pi}" upper="${pi}" velocity="10.0" effort="10.0"/>
 	</joint>
+	<transmission name="hip_transmission">
+		<type>transmission_interface/SimpleTransmission</type>
+		<joint name="hip_joint">
+			<hardwareInterface>hardware_interface/PositionJointInterface</hardwareInterface>
+		</joint>
+		<actuator name="hip_motor">
+			<hardwareInterface>hardware_interface/PositionJointInterface</hardwareInterface>
+			<mechanicalReduction>1</mechanicalReduction>
+		</actuator>
+	</transmission>
+	<transmission name="shoulder_transmission">
+		<type>transmission_interface/SimpleTransmission</type>
+		<joint name="shoulder_joint">
+			<hardwareInterface>hardware_interface/PositionJointInterface</hardwareInterface>
+		</joint>
+		<actuator name="shoulder_motor">
+			<hardwareInterface>hardware_interface/PositionJointInterface</hardwareInterface>
+			<mechanicalReduction>1</mechanicalReduction>
+		</actuator>
+	</transmission>
+	<transmission name="elbow_transmission">
+		<type>transmission_interface/SimpleTransmission</type>
+		<joint name="elbow_joint">
+			<hardwareInterface>hardware_interface/PositionJointInterface</hardwareInterface>
+		</joint>
+		<actuator name="elbow_motor">
+			<hardwareInterface>hardware_interface/PositionJointInterface</hardwareInterface>
+			<mechanicalReduction>1</mechanicalReduction>
+		</actuator>
+	</transmission>
 	<gazebo>
 		<static>false</static>

Commit message: Wrist joint, need to add gripper

File: urdf/roboarm.urdf.xacro (robot description, xacro)
@@ -14,4 +14,6 @@
 	<xacro:property name="elbow_length" value="0.9"/>
 	<xacro:property name="elbow_radius" value="0.1"/>
+	<xacro:property name="wrist_mass" value="1.0"/>
+	<xacro:property name="wrist_radius" value="0.05"/>
 	<xacro:property name="pi" value="3.141492653589793"/>
 	<link name="world"/>
@@ -111,4 +113,52 @@
 			</geometry>
 		</collision>
+	</link>
+	<link name="wrist_yaw_link">
+		<inertial>
+			<mass value="${wrist_mass}"/>
+			<origin xyz="0 0 0" rpy="0 0 0"/>
+			<inertia ixx="${2*wrist_mass*wrist_radius*wrist_radius/5}"
+					 ixy="0.0"
+					 ixz="0.0"
+					 iyy="${2*wrist_mass*wrist_radius*wrist_radius/5}"
+					 iyz="0.0"
+					 izz="${2*wrist_mass*wrist_radius*wrist_radius/5}"/>
+		</inertial>
+		<visual name="wrist_yaw_link_visual">
+			<origin xyz="0 0 0" rpy="0 0 0"/>
+			<geometry>
+				<sphere radius="${wrist_radius}"/>
+			</geometry>
+		</visual>
+		<collision name="wrist_yaw_link_collision">
+			<origin xyz="0 0 0" rpy="0 0 0"/>
+			<geometry>
+				<sphere radius="${wrist_radius}"/>
+			</geometry>
+		</collision>
+	</link>
+	<link name="wrist_pitch_link">
+		<inertial>
+			<mass value="${wrist_mass}"/>
+			<origin xyz="0 0 0" rpy="0 0 0"/>
+			<inertia ixx="${2*wrist_mass*wrist_radius*wrist_radius/5}"
+					 ixy="0.0"
+					 ixz="0.0"
+					 iyy="${2*wrist_mass*wrist_radius*wrist_radius/5}"
+					 iyz="0.0"
+					 izz="${2*wrist_mass*wrist_radius*wrist_radius/5}"/>
+		</inertial>
+	</link>
+	<link name="wrist_roll_link">
+		<inertial>
+			<mass value="${wrist_mass}"/>
+			<origin xyz="0 0 0" rpy="0 0 0"/>
+			<inertia ixx="${2*wrist_mass*wrist_radius*wrist_radius/5}"
+					 ixy="0.0"
+					 ixz="0.0"
+					 iyy="${2*wrist_mass*wrist_radius*wrist_radius/5}"
+					 iyz="0.0"
+					 izz="${2*wrist_mass*wrist_radius*wrist_radius/5}"/>
+		</inertial>
 	</link>
 	<joint name="world_joint" type="fixed">
@@ -136,4 +186,24 @@
 		<limit lower="${-pi}" upper="${pi}" velocity="10.0" effort="10.0"/>
 	</joint>
+	<joint name="wrist_yaw_joint" type="revolute">
+		<parent link="elbow_link"/>
+		<child link="wrist_yaw_link"/>
+		<origin xyz="0 0 ${elbow_length-elbow_radius}" rpy="0 0 0"/>
+		<axis xyz="0 1 0"/>
+		<limit lower="${-pi/2}" upper="${pi/2}" velocity="10.0" effort="10.0"/>
+	</joint>
+	<joint name="wrist_pitch_joint" type="revolute">
+		<parent link="wrist_yaw_link"/>
+		<child link="wrist_pitch_link"/>
+		<origin xyz="0 0 0" rpy="0 0 0"/>
+		<axis xyz="1 0 0"/>
+		<limit lower="${-pi/2}" upper="${pi/2}" velocity="10.0" effort="10.0"/>
+	</joint>
+	<joint name="wrist_roll_joint" type="continuous">
+		<parent link="wrist_pitch_link"/>
+		<child link="wrist_roll_link"/>
+		<origin xyz="0 0 0" rpy="0 0 0"/>
+		<axis xyz="0 0 1"/>
+	</joint>
 	<transmission name="hip_transmission">
 		<type>transmission_interface/SimpleTransmission</type>
@@ -162,4 +232,34 @@
 		</joint>
 		<actuator name="elbow_motor">
+			<hardwareInterface>hardware_interface/PositionJointInterface</hardwareInterface>
+			<mechanicalReduction>1</mechanicalReduction>
+		</actuator>
+	</transmission>
+	<transmission name="wrist_yaw_transmission">
+		<type>transmission_interface/SimpleTransmission</type>
+		<joint name="wrist_yaw_joint">
+			<hardwareInterface>hardware_interface/PositionJointInterface</hardwareInterface>
+		</joint>
+		<actuator name="wrist_yaw_motor">
+			<hardwareInterface>hardware_interface/PositionJointInterface</hardwareInterface>
+			<mechanicalReduction>1</mechanicalReduction>
+		</actuator>
+	</transmission>
+	<transmission name="wrist_pitch_transmission">
+		<type>transmission_interface/SimpleTransmission</type>
+		<joint name="wrist_pitch_joint">
+			<hardwareInterface>hardware_interface/PositionJointInterface</hardwareInterface>
+		</joint>
+		<actuator name="wrist_pitch_motor">
+			<hardwareInterface>hardware_interface/PositionJointInterface</hardwareInterface>
+			<mechanicalReduction>1</mechanicalReduction>
+		</actuator>
+	</transmission>
+	<transmission name="wrist_roll_transmission">
+		<type>transmission_interface/SimpleTransmission</type>
+		<joint name="wrist_roll_joint">
+			<hardwareInterface>hardware_interface/PositionJointInterface</hardwareInterface>
+		</joint>
+		<actuator name="wrist_roll_motor">
 			<hardwareInterface>hardware_interface/PositionJointInterface</hardwareInterface>
 			<mechanicalReduction>1</mechanicalReduction>
@@ -172,5 +272,5 @@
 		</plugin>
 		<plugin name="joint_state_publisher" filename="libgazebo_ros_joint_state_publisher.so">
-			<jointName>hip_joint, shoulder_joint, elbow_joint</jointName>
+			<jointName>hip_joint, shoulder_joint, elbow_joint, wrist_yaw_joint, wrist_pitch_joint, wrist_roll_joint</jointName>
 			<robotNamespace>/roboarm</robotNamespace>
 		</plugin>

Commit message: Added gripper

File: urdf/roboarm.urdf.xacro (robot description, xacro)
@@ -16,5 +16,8 @@
 	<xacro:property name="wrist_mass" value="1.0"/>
 	<xacro:property name="wrist_radius" value="0.05"/>
-	<xacro:property name="pi" value="3.141492653589793"/>
+	<xacro:property name="gripper_mass" value="0.1"/>
+	<xacro:property name="gripper_height" value="0.01"/>
+	<xacro:property name="gripper_length" value="0.2"/>
+	<xacro:property name="gripper_width" value="0.025"/>
 	<link name="world"/>
 	<link name="base_link">
@@ -161,4 +164,100 @@
 					 izz="${2*wrist_mass*wrist_radius*wrist_radius/5}"/>
 		</inertial>
+	</link>
+	<link name="gripper_lower_right_link">
+		<inertial>
+			<mass value="${gripper_mass}"/>
+			<origin xyz="0 0 0" rpy="0 0 0"/>
+			<inertia ixx="0.0"
+					 ixy="0.0"
+					 ixz="0.0"
+					 iyy="0.0"
+					 iyz="0.0"
+					 izz="0.0"/>
+		</inertial>
+		<visual name="gripper_lower_right_link_visual">
+			<origin xyz="${gripper_length*cos(pi/4)/2} 0 ${gripper_length*sin(pi/4)/2}" rpy="0 ${pi/4} 0"/>
+			<geometry>
+				<box size="${gripper_height} ${gripper_width} ${gripper_length}"/>
+			</geometry>
+		</visual>
+		<collision name="gripper_lower_right_link_collision">
+			<origin xyz="${gripper_length*cos(pi/4)/2} 0 ${gripper_length*sin(pi/4)/2}" rpy="0 ${pi/4} 0"/>
+			<geometry>
+				<box size="${gripper_height} ${gripper_width} ${gripper_length}"/>
+			</geometry>
+		</collision>
+	</link>
+	<link name="gripper_lower_left_link">
+		<inertial>
+			<mass value="${gripper_mass}"/>
+			<origin xyz="0 0 0" rpy="0 0 0"/>
+			<inertia ixx="0.0"
+					 ixy="0.0"
+					 ixz="0.0"
+					 iyy="0.0"
+					 iyz="0.0"
+					 izz="0.0"/>
+		</inertial>
+		<visual name="gripper_lower_left_link_visual">
+			<origin xyz="${-gripper_length*cos(pi/4)/2} 0 ${gripper_length*sin(pi/4)/2}" rpy="0 ${-pi/4} 0"/>
+			<geometry>
+				<box size="${gripper_height} ${gripper_width} ${gripper_length}"/>
+			</geometry>
+		</visual>
+		<collision name="gripper_lower_left_link_collision">
+			<origin xyz="${-gripper_length*cos(pi/4)/2} 0 ${gripper_length*sin(pi/4)/2}" rpy="0 ${-pi/4} 0"/>
+			<geometry>
+				<box size="${gripper_height} ${gripper_width} ${gripper_length}"/>
+			</geometry>
+		</collision>
+	</link>
+	<link name="gripper_upper_right_link">
+		<inertial>
+			<mass value="${gripper_mass}"/>
+			<origin xyz="0 0 0" rpy="0 0 0"/>
+			<inertia ixx="0.0"
+					 ixy="0.0"
+					 ixz="0.0"
+					 iyy="0.0"
+					 iyz="0.0"
+					 izz="0.0"/>
+		</inertial>
+		<visual name="gripper_upper_right_link_visual">
+			<origin xyz="0 0 ${gripper_length/2}" rpy="0 0 0"/>
+			<geometry>
+				<box size="${gripper_height} ${gripper_width} ${gripper_length}"/>
+			</geometry>
+		</visual>
+		<collision name="gripper_upper_right_link_collision">
+			<origin xyz="0 0 ${gripper_length/2}" rpy="0 0 0"/>
+			<geometry>
+				<box size="${gripper_height} ${gripper_width} ${gripper_length}"/>
+			</geometry>
+		</collision>
+	</link>
+	<link name="gripper_upper_left_link">
+		<inertial>
+			<mass value="${gripper_mass}"/>
+			<origin xyz="0 0 0" rpy="0 0 0"/>
+			<inertia ixx="0.0"
+					 ixy="0.0"
+					 ixz="0.0"
+					 iyy="0.0"
+					 iyz="0.0"
+					 izz="0.0"/>
+		</inertial>
+		<visual name="gripper_upper_left_link_visual">
+			<origin xyz="0 0 ${gripper_length/2}" rpy="0 0 0"/>
+			<geometry>
+				<box size="${gripper_height} ${gripper_width} ${gripper_length}"/>
+			</geometry>
+		</visual>
+		<collision name="gripper_upper_left_link_collision">
+			<origin xyz="0 0 ${gripper_length/2}" rpy="0 0 0"/>
+			<geometry>
+				<box size="${gripper_height} ${gripper_width} ${gripper_length}"/>
+			</geometry>
+		</collision>
 	</link>
 	<joint name="world_joint" type="fixed">
@@ -206,4 +305,32 @@
 		<axis xyz="0 0 1"/>
 	</joint>
+	<joint name="gripper_lower_left_joint" type="revolute">
+		<parent link="wrist_roll_link"/>
+		<child link="gripper_lower_left_link"/>
+		<origin xyz="0 0 0" rpy="0 0 0"/>
+		<axis xyz="0 1 0"/>
+		<limit lower="0.0" upper="${pi/4}" velocity="10.0" effort="10.0"/>
+	</joint>
+	<joint name="gripper_lower_right_joint" type="revolute">
+		<parent link="wrist_roll_link"/>
+		<child link="gripper_lower_right_link"/>
+		<origin xyz="0 0 0" rpy="0 0 0"/>
+		<axis xyz="0 1 0"/>
+		<limit lower="0.0" upper="${pi/4}" velocity="10.0" effort="10.0"/>
+	</joint>
+	<joint name="gripper_upper_left_joint" type="revolute">
+		<parent link="gripper_lower_left_link"/>
+		<child link="gripper_upper_left_link"/>
+		<origin xyz="${gripper_length*cos(pi/4)} 0 ${gripper_length*sin(pi/4)}" rpy="0 0 0"/>
+		<axis xyz="0 1 0"/>
+		<limit lower="0.0" upper="${pi/4}" velocity="10.0" effort="10.0"/>
+	</joint>
+	<joint name="gripper_upper_right_joint" type="revolute">
+		<parent link="gripper_lower_right_link"/>
+		<child link="gripper_upper_right_link"/>
+		<origin xyz="${-gripper_length*cos(pi/4)} 0 ${gripper_length*sin(pi/4)}" rpy="0 0 0"/>
+		<axis xyz="0 1 0"/>
+		<limit lower="0.0" upper="${pi/4}" velocity="10.0" effort="10.0"/>
+	</joint>
 	<transmission name="hip_transmission">
 		<type>transmission_interface/SimpleTransmission</type>
@@ -272,5 +399,6 @@
 		</plugin>
 		<plugin name="joint_state_publisher" filename="libgazebo_ros_joint_state_publisher.so">
-			<jointName>hip_joint, shoulder_joint, elbow_joint, wrist_yaw_joint, wrist_pitch_joint, wrist_roll_joint</jointName>
+			<jointName>hip_joint, shoulder_joint, elbow_joint, wrist_yaw_joint, wrist_pitch_joint, wrist_roll_joint,
+				gripper_lower_left_joint, gripper_lower_right_joint, gripper_upper_left_joint, gripper_upper_right_joint</jointName>
 			<robotNamespace>/roboarm</robotNamespace>
 		</plugin>

Commit message: Mimic joints for gripper

File: urdf/roboarm.urdf.xacro (robot description, xacro)
@@ -18,5 +18,5 @@
 	<xacro:property name="gripper_mass" value="0.1"/>
 	<xacro:property name="gripper_height" value="0.01"/>
-	<xacro:property name="gripper_length" value="0.2"/>
+	<xacro:property name="gripper_length" value="0.1"/>
 	<xacro:property name="gripper_width" value="0.025"/>
 	<link name="world"/>
@@ -310,5 +310,5 @@
 		<origin xyz="0 0 0" rpy="0 0 0"/>
 		<axis xyz="0 1 0"/>
-		<limit lower="0.0" upper="${pi/4}" velocity="10.0" effort="10.0"/>
+		<limit lower="0.0" upper="${pi/5}" velocity="1.0" effort="10.0"/>
 	</joint>
 	<joint name="gripper_lower_right_joint" type="revolute">
@@ -317,19 +317,19 @@
 		<origin xyz="0 0 0" rpy="0 0 0"/>
 		<axis xyz="0 1 0"/>
-		<limit lower="0.0" upper="${pi/4}" velocity="10.0" effort="10.0"/>
+		<limit lower="${-pi/5}" upper="0.0" velocity="1.0" effort="10.0"/>
 	</joint>
 	<joint name="gripper_upper_left_joint" type="revolute">
 		<parent link="gripper_lower_left_link"/>
 		<child link="gripper_upper_left_link"/>
-		<origin xyz="${gripper_length*cos(pi/4)} 0 ${gripper_length*sin(pi/4)}" rpy="0 0 0"/>
+		<origin xyz="${-gripper_length*cos(pi/4)} 0 ${gripper_length*sin(pi/4)}" rpy="0 0 0"/>
 		<axis xyz="0 1 0"/>
-		<limit lower="0.0" upper="${pi/4}" velocity="10.0" effort="10.0"/>
+		<limit lower="${-pi/5}" upper="0.0" velocity="1.0" effort="10.0"/>
 	</joint>
 	<joint name="gripper_upper_right_joint" type="revolute">
 		<parent link="gripper_lower_right_link"/>
 		<child link="gripper_upper_right_link"/>
-		<origin xyz="${-gripper_length*cos(pi/4)} 0 ${gripper_length*sin(pi/4)}" rpy="0 0 0"/>
+		<origin xyz="${gripper_length*cos(pi/4)} 0 ${gripper_length*sin(pi/4)}" rpy="0 0 0"/>
 		<axis xyz="0 1 0"/>
-		<limit lower="0.0" upper="${pi/4}" velocity="10.0" effort="10.0"/>
+		<limit lower="0.0" upper="${pi/5}" velocity="1.0" effort="10.0"/>
 	</joint>
 	<transmission name="hip_transmission">
@@ -389,4 +389,44 @@
 		</joint>
 		<actuator name="wrist_roll_motor">
+			<hardwareInterface>hardware_interface/PositionJointInterface</hardwareInterface>
+			<mechanicalReduction>1</mechanicalReduction>
+		</actuator>
+	</transmission>
+	<transmission name="gripper_lower_left_transmission">
+		<type>transmission_interface/SimpleTransmission</type>
+		<joint name="gripper_lower_left_joint">
+			<hardwareInterface>hardware_interface/PositionJointInterface</hardwareInterface>
+		</joint>
+		<actuator name="gripper_lower_left_motor">
+			<hardwareInterface>hardware_interface/PositionJointInterface</hardwareInterface>
+			<mechanicalReduction>1</mechanicalReduction>
+		</actuator>
+	</transmission>
+	<transmission name="gripper_lower_right_transmission">
+		<type>transmission_interface/SimpleTransmission</type>
+		<joint name="gripper_lower_right_joint">
+			<hardwareInterface>hardware_interface/PositionJointInterface</hardwareInterface>
+		</joint>
+		<actuator name="gripper_lower_right_motor">
+			<hardwareInterface>hardware_interface/PositionJointInterface</hardwareInterface>
+			<mechanicalReduction>1</mechanicalReduction>
+		</actuator>
+	</transmission>
+	<transmission name="gripper_upper_left_transmission">
+		<type>transmission_interface/SimpleTransmission</type>
+		<joint name="gripper_upper_left_joint">
+			<hardwareInterface>hardware_interface/PositionJointInterface</hardwareInterface>
+		</joint>
+		<actuator name="gripper_upper_left_motor">
+			<hardwareInterface>hardware_interface/PositionJointInterface</hardwareInterface>
+			<mechanicalReduction>1</mechanicalReduction>
+		</actuator>
+	</transmission>
+	<transmission name="gripper_upper_right_transmission">
+		<type>transmission_interface/SimpleTransmission</type>
+		<joint name="gripper_upper_right_joint">
+			<hardwareInterface>hardware_interface/PositionJointInterface</hardwareInterface>
+		</joint>
+		<actuator name="gripper_upper_right_motor">
 			<hardwareInterface>hardware_interface/PositionJointInterface</hardwareInterface>
 			<mechanicalReduction>1</mechanicalReduction>
@@ -403,4 +443,25 @@
 			<robotNamespace>/roboarm</robotNamespace>
 		</plugin>
+		<plugin name = "lower_right_mimic_joint" filename = "libroboticsgroup_gazebo_mimic_joint_plugin.so">
+			<robotNamespace> /roboarm </robotNamespace>
+			<joint> gripper_lower_left_joint </joint>
+			<mimicJoint> gripper_lower_right_joint </mimicJoint>
+			<multiplier> -1 </multiplier>
+			<offset> 0 </offset>
+		</plugin>
+		<plugin name = "upper_left_mimic_joint" filename = "libroboticsgroup_gazebo_mimic_joint_plugin.so">
+			<robotNamespace> /roboarm </robotNamespace>
+			<joint> gripper_lower_left_joint </joint>
+			<mimicJoint> gripper_upper_left_joint </mimicJoint>
+			<multiplier> -0.8 </multiplier>
+			<offset> 0 </offset>
+		</plugin>
+		<plugin name = "upper_right_mimic_joint" filename = "libroboticsgroup_gazebo_mimic_joint_plugin.so">
+			<robotNamespace> /roboarm </robotNamespace>
+			<joint> gripper_lower_left_joint </joint>
+			<mimicJoint> gripper_upper_right_joint </mimicJoint>
+			<multiplier> 0.8 </multiplier>
+			<offset> 0 </offset>
+		</plugin>
 	</gazebo>
 </robot>

Commit message: Using gazebo_grasph_plugin

File: urdf/roboarm.urdf.xacro (robot description, xacro)
@@ -261,4 +261,5 @@
 		</collision>
 	</link>
+	<link name="gripper"/>
 	<joint name="world_joint" type="fixed">
 		<parent link="world"/>
@@ -333,4 +334,8 @@
 		<limit lower="0.0" upper="${pi/5}" velocity="1.0" effort="10.0"/>
 	</joint>
+	<joint name="gripper_joint" type="fixed">
+		<parent link="wrist_roll_link"/>
+		<child link="gripper"/>
+	</joint>
 	<transmission name="hip_transmission">
 		<type>transmission_interface/SimpleTransmission</type>
@@ -454,5 +459,5 @@
 			<joint> gripper_lower_left_joint </joint>
 			<mimicJoint> gripper_upper_left_joint </mimicJoint>
-			<multiplier> -0.8 </multiplier>
+			<multiplier> -1 </multiplier>
 			<offset> 0 </offset>
 		</plugin>
@@ -461,6 +466,23 @@
 			<joint> gripper_lower_left_joint </joint>
 			<mimicJoint> gripper_upper_right_joint </mimicJoint>
-			<multiplier> 0.8 </multiplier>
+			<multiplier> 1 </multiplier>
 			<offset> 0 </offset>
+		</plugin>
+		<plugin name="gazebo_grasp_fix" filename="libgazebo_grasp_fix.so">
+			<arm>
+				<arm_name>roboarm</arm_name>
+				<palm_link> wrist_roll_link  </palm_link>
+				<gripper_link> gripper_lower_left_link </gripper_link>
+				<gripper_link> gripper_lower_right_link </gripper_link>
+				<gripper_link> gripper_upper_left_link </gripper_link>
+				<gripper_link> gripper_upper_right_link </gripper_link>
+			</arm>
+			<forces_angle_tolerance>100</forces_angle_tolerance>
+			<update_rate>4</update_rate>
+			<grip_count_threshold>4</grip_count_threshold>
+			<max_grip_count>8</max_grip_count>
+			<release_tolerance>0.005</release_tolerance>
+			<disable_collisions_on_attach>false</disable_collisions_on_attach>
+			<contact_topic>__default_topic__</contact_topic>
 		</plugin>
 	</gazebo>

Commit message: Added Kinect link to roboarm, will use plugin for autonomous operation

File: urdf/roboarm.urdf.xacro (robot description, xacro)
@@ -3,6 +3,6 @@
 	<xacro:property name="base_mass" value="100.0"/>
 	<xacro:property name="base_height" value="0.1"/>
-	<xacro:property name="base_length" value="0.25"/>
-	<xacro:property name="base_width" value="0.25"/>
+	<xacro:property name="base_length" value="0.35"/>
+	<xacro:property name="base_width" value="0.35"/>
 	<xacro:property name="hip_mass" value="10.0"/>
 	<xacro:property name="hip_length" value="1.0"/>
@@ -20,4 +20,7 @@
 	<xacro:property name="gripper_length" value="0.1"/>
 	<xacro:property name="gripper_width" value="0.025"/>
+	<xacro:property name="kinect_height" value="0.072"/>
+	<xacro:property name="kinect_length" value="0.276"/>
+	<xacro:property name="kinect_width" value="0.073"/>
 	<link name="world"/>
 	<link name="base_link">
@@ -262,7 +265,20 @@
 	</link>
 	<link name="gripper"/>
+	<link name="kinect_link">
+		<visual>
+			<origin xyz = "0 0 0"/>
+			<geometry>
+				<mesh filename="package://roboarm/meshes/kinect.dae"/>
+			</geometry>
+		</visual>
+	</link>
 	<joint name="world_joint" type="fixed">
 		<parent link="world"/>
 		<child link="base_link"/>
+	</joint>
+	<joint name="kinect_fixed" type="fixed">
+		<parent link="base_link"/>
+		<child link="kinect_link"/>
+		<origin xyz = "0 ${base_length/2} ${base_height+kinect_height/2}" rpy="0 0 ${pi/2}"/>
 	</joint>
 	<joint name="hip_joint" type="continuous">

Commit message: Added Kinect sensor with plugin to model base

File: urdf/roboarm.urdf.xacro (robot description, xacro)
@@ -266,4 +266,14 @@
 	<link name="gripper"/>
 	<link name="kinect_link">
+		<inertial>
+			<mass value="0.1"/>
+			<origin xyz="0 0 0"/>
+			<inertia ixx="0.0"
+					 ixy="0.0"
+					 ixz="0.0"
+					 iyy="0.0"
+					 iyz="0.0"
+					 izz="0.0"/>
+		</inertial>
 		<visual>
 			<origin xyz = "0 0 0"/>
@@ -277,8 +287,9 @@
 		<child link="base_link"/>
 	</joint>
-	<joint name="kinect_fixed" type="fixed">
+	<joint name="kinect_joint" type="revolute">
 		<parent link="base_link"/>
 		<child link="kinect_link"/>
-		<origin xyz = "0 ${base_length/2} ${base_height+kinect_height/2}" rpy="0 0 ${pi/2}"/>
+		<origin xyz = "0 ${base_length/2} ${base_height+kinect_height/2+0.02}" rpy="0 0 ${pi/2}"/>
+		<limit lower="-0.1" upper="0.1" effort="1.0" velocity="1.0"/>
 	</joint>
 	<joint name="hip_joint" type="continuous">
@@ -503,3 +514,48 @@
 		</plugin>
 	</gazebo>
+	<gazebo reference="kinect_link">
+		<sensor type="depth" name="depth_sensor">
+			<update_rate>30.0</update_rate>
+			<camera name="kinect">
+				<horizontal_fov>1.3962634</horizontal_fov>
+				<image>
+					<width>1280</width>
+					<height>1024</height>
+					<format>R8G8B8</format>
+				</image>
+				<clip>
+					<near>0.02</near>
+					<far>300</far>
+				</clip>
+				<noise>
+					<type>gaussian</type>
+					<mean>0.0</mean>
+					<stddev>0.007</stddev>
+				</noise>
+			</camera>
+			<plugin name="kinect" filename="libgazebo_ros_openni_kinect.so">
+				<baseline>0.2</baseline>
+				<alwaysOn>true</alwaysOn>
+				<updateRate>30.0</updateRate>
+				<cameraName>kinect</cameraName>
+				<imageTopicName>/kinect/depth/image_raw</imageTopicName>
+				<cameraInfoTopicName>/kinect/depth/camera_info</cameraInfoTopicName>
+				<depthImageTopicName>/kinect/depth/image_raw</depthImageTopicName>
+				<depthImageInfoTopicName>/kinect/depth/camera_info</depthImageInfoTopicName>
+				<pointCloudTopicName>/kinect/depth/points</pointCloudTopicName>
+				<frameName>base_link</frameName>
+				<pointCloudCutoff>0.5</pointCloudCutoff>
+				<distortionK1>0.00000001</distortionK1>
+				<distortionK2>0.00000001</distortionK2>
+				<distortionK3>0.00000001</distortionK3>
+				<distortionT1>0.00000001</distortionT1>
+				<distortionT2>0.00000001</distortionT2>
+				<CxPrime>0</CxPrime>
+				<Cx>0</Cx>
+				<Cy>0</Cy>
+				<focalLength>0</focalLength>
+				<hackBaseline>0</hackBaseline>
+			</plugin>
+		</sensor>
+	</gazebo>
 </robot>
